Commit message: feat: add LDS-01 LiDAR to URDF

File: ros2_ws/src/burgerbot_bringup/urdf/burger_robot.urdf (robot description, URDF)
Before this commit: robot burger_robot, 7 links, 6 joints
Links:
- added link base_scan, mass 0.114; collision cylinder length=0.055 radius=0.0508; visual cylinder length=0.055 radius=0.0508
Joints:
- added joint scan_joint: type fixed, parent base_link, child base_scan, origin xyz=-0.032 0 0.171 rpy=0 0 0
