Commit message: firmware: one-shot kickstart PWM=60/200ms, FF=0.8, Ki=1.0, timeout=1000ms, no PID reset. nav2: linear_vel 0.35, no collision detect, map path, bond_timeout 4.0. ekf: no vyaw, zero gyro bias. rviz: map/plan/costmap/particles displays. imu tf disabled. wheel radius corrected

File: ros2_ws/src/rep_description/urdf/assemblies/rep.urdf.xacro (robot description, xacro)
@@ -192,4 +192,10 @@
       <origin xyz="-0.000000 -0.000000 0.075500" rpy="-0.000000 0.000000 0.000000"/>
     </joint>
+    <link name="${prefix}imu_link"/>
+    <joint name="${prefix}imu_link_joint" type="fixed">
+      <parent link="${prefix}imu"/>
+      <child link="${prefix}imu_link"/>
+      <origin xyz="0 0 0" rpy="0 0 0"/>
+    </joint>
     <joint name="${prefix}mag_joint" type="fixed">
       <parent link="${prefix}base_link"/>
@@ -200,5 +206,5 @@
       <parent link="${prefix}base_link"/>
       <child link="${prefix}left_wheel"/>
-      <origin xyz="-0.000000 0.119500 -0.027000" rpy="0.000000 -0.000000 -0.000000"/>
+      <origin xyz="-0.000000 0.141000 -0.027000" rpy="0.000000 -0.000000 -0.000000"/>
       <axis xyz="-0.000000 1.000000 -0.000000"/>
       <limit effort="100.0" velocity="1.00"/>
@@ -207,5 +213,5 @@
       <parent link="${prefix}base_link"/>
       <child link="${prefix}right_wheel"/>
-      <origin xyz="-0.000000 -0.119500 -0.027000" rpy="-0.000000 -0.000000 -0.000000"/>
+      <origin xyz="-0.000000 -0.141000 -0.027000" rpy="-0.000000 -0.000000 -0.000000"/>
       <axis xyz="0.000000 -1.000000 -0.000000"/>
       <limit effort="100.0" velocity="1.00"/>

File: ros2_ws/src/rep_description/urdf/rep.urdf (robot description, URDF)
Before this commit: robot rep, 9 links, 8 joints
Joints:
- joint left_wheel_joint: origin xyz=-0.000000 0.119500 -0.027000 rpy=0.000000 -0.000000 -0.000000 -> xyz=-0.000000 0.141000 -0.027000 rpy=0.000000 -0.000000 -0.000000
- joint right_wheel_joint: origin xyz=-0.000000 -0.119500 -0.027000 rpy=-0.000000 -0.000000 -0.000000 -> xyz=-0.000000 -0.141000 -0.027000 rpy=-0.000000 -0.000000 -0.000000
