Commit message: fix(urdf): remove pi property redefinition
xacro in ROS2 Jazzy provides pi as a built-in constant.
Defining it again emits a stderr warning that causes Command()
in launch files to throw an exception.

Co-Authored-By: Claude Sonnet 4.6 <noreply@anthropic.com>

File: ros2_ws/src/burgerbot/urdf/burgerbot.urdf.xacro (robot description, xacro)
@@ -11,5 +11,4 @@
   <xacro:property name="lidar_z"          value="0.171"/>
   <xacro:property name="imu_z"            value="0.050"/>
-  <xacro:property name="pi"               value="3.14159265358979"/>
   <!-- ── Materials ── -->
   <material name="chassis_grey"><color rgba="0.65 0.65 0.65 1.0"/></material>
